Commit message: core.launch.py in main launch for robot package

File: src/my_robot_description/urdf/robot_core.xacro (robot description, xacro)
@@ -23,5 +23,5 @@
       <origin xyz="0 0 0" rpy="0 -0.0 0"/>
       <geometry>
-        <mesh filename="package://my_robot_description/meshes/visual/sejongDel_body_origin45.dae" scale="0.00075 0.00075 0.00075"/>
+        <mesh filename="package://my_robot_description/meshes/visual/sejongDel_body_origin45.dae" scale="0.00075 0.0005 0.00075"/>
       </geometry>
     </visual>
@@ -29,5 +29,5 @@
       <origin xyz="0 0 0" rpy="0 -0.0 0"/>
       <geometry>
-        <mesh filename="package://my_robot_description/meshes/collision/sejongDel_body_origin45.stl" scale="0.00075 0.00075 0.00075"/>
+        <mesh filename="package://my_robot_description/meshes/collision/sejongDel_body_origin45.stl" scale="0.00075 0.0005 0.00075"/>
       </geometry>
     </collision>
@@ -60,5 +60,5 @@
     <parent link="base_link"/>
     <child link="left_wheel"/>
-    <origin xyz="${0.28-wheel_radius} ${wheel_separation/2} 0.3" rpy="0 0 0"/>
+    <origin xyz="${0.28-wheel_radius} ${wheel_separation/2-0.1} 0.3" rpy="0 0 0"/>
     <axis xyz="0 1 0"/>
   </joint>
@@ -85,5 +85,5 @@
     <parent link="base_link"/>
     <child link="right_wheel"/>
-    <origin xyz="${0.28-wheel_radius} -${wheel_separation/2} 0.3" rpy="0 0 0"/>
+    <origin xyz="${0.28-wheel_radius} -${wheel_separation/2-0.1} 0.3" rpy="0 0 0"/>
     <axis xyz="0 1 0"/>
   </joint>

Commit message: update: core.launch.py, robot_core.xacro

File: src/my_robot_description/urdf/robot_core.xacro (robot description, xacro)
@@ -52,5 +52,5 @@
     </collision>
     <inertial>
-      <mass value="1.0"/>
+      <mass value="0.5"/>
       <inertia ixx="0.01" ixy="0.0" ixz="0.0" iyy="0.01" iyz="0.0" izz="0.01"/>
       <origin xyz="0 0 0"/>
@@ -77,5 +77,5 @@
     </collision>
     <inertial>
-      <mass value="1.0"/>
+      <mass value="0.5"/>
       <inertia ixx="0.01" ixy="0.0" ixz="0.0" iyy="0.01" iyz="0.0" izz="0.01"/>
       <origin xyz="0 0 0"/>
@@ -102,5 +102,5 @@
     </collision>
     <inertial>
-      <mass value="1.0"/>
+      <mass value="0.5"/>
       <inertia ixx="0.01" ixy="0.0" ixz="0.0" iyy="0.01" iyz="0.0" izz="0.01"/>
       <origin xyz="0 0 0"/>
@@ -135,5 +135,5 @@
     <parent link="base_link"/>
     <child link="front_camera"/>
-    <origin xyz="0.3 0 0.6" rpy="0 -${pi/4} 0"/>
+    <origin xyz="0.3 0 0.25" rpy="0 -${pi/4+0.17453/2} 0"/>
   </joint>
   <gazebo reference="front_camera">

Commit message: edit something

File: src/my_robot_description/urdf/robot_core.xacro (robot description, xacro)
@@ -33,6 +33,6 @@
     </collision>
     <inertial>
-      <mass value="0.1"/>
-      <inertia ixx="0.01" ixy="0.0" ixz="0.0" iyy="0.01" iyz="0.0" izz="0.01"/>
+      <mass value="0.01"/>
+      <inertia ixx="0.001" ixy="0.0" ixz="0.0" iyy="0.001" iyz="0.0" izz="0.001"/>
       <origin xyz="0 0 0"/>
     </inertial>
@@ -60,5 +60,5 @@
     <parent link="base_link"/>
     <child link="left_wheel"/>
-    <origin xyz="${0.28-wheel_radius} ${wheel_separation/2-0.1} 0.3" rpy="0 0 0"/>
+    <origin xyz="${0.28-wheel_radius} ${wheel_separation/2-0.05} 0.3" rpy="0 0 0"/>
     <axis xyz="0 1 0"/>
   </joint>
@@ -85,12 +85,12 @@
     <parent link="base_link"/>
     <child link="right_wheel"/>
-    <origin xyz="${0.28-wheel_radius} -${wheel_separation/2-0.1} 0.3" rpy="0 0 0"/>
+    <origin xyz="${0.28-wheel_radius} -${wheel_separation/2-0.05} 0.3" rpy="0 0 0"/>
     <axis xyz="0 1 0"/>
   </joint>
-  <link name="rear_wheel">
+  <link name="left_rear_wheel">
     <visual>
       <origin xyz="0 0 0" rpy="0 0 ${pi/2}"/>
       <geometry>
-        <mesh filename="package://my_robot_description/meshes/visual/wheel.dae" scale="2 2 2"/>
+        <mesh filename="package://my_robot_description/meshes/visual/wheel.dae" scale="5 5 5"/>
       </geometry>
     </visual>
@@ -98,18 +98,45 @@
       <origin xyz="0 0 0" rpy="0 0 ${pi/2}"/>
       <geometry>
-        <mesh filename="package://my_robot_description/meshes/collision/wheel.stl" scale="2 2 2"/>
+        <mesh filename="package://my_robot_description/meshes/collision/wheel.stl" scale="5 5 5"/>
       </geometry>
     </collision>
     <inertial>
-      <mass value="0.5"/>
+      <mass value="0.25"/>
       <inertia ixx="0.01" ixy="0.0" ixz="0.0" iyy="0.01" iyz="0.0" izz="0.01"/>
       <origin xyz="0 0 0"/>
     </inertial>
   </link>
-  <joint name="rear_wheel_joint" type="continuous">
+  <joint name="left_rear_wheel_joint" type="continuous">
     <parent link="base_link"/>
-    <child link="rear_wheel"/>
-    <origin xyz="-${0.1+wheel_radius-0.15} 0 -0.1" rpy="0 0 0"/>
+    <child link="left_rear_wheel"/>
+    <origin xyz="-${0.28-wheel_radius+0.05} ${wheel_separation/2-0.05} -0.1" rpy="0 0 0"/>
     <axis xyz="0 1 0"/>
+    <dynamics friction="0.0" damping="0.0"/>
+  </joint>
+  <link name="right_rear_wheel">
+    <visual>
+      <origin xyz="0 0 0" rpy="0 0 ${pi/2}"/>
+      <geometry>
+        <mesh filename="package://my_robot_description/meshes/visual/wheel.dae" scale="5 5 5"/>
+      </geometry>
+    </visual>
+    <collision>
+      <origin xyz="0 0 0" rpy="0 0 ${pi/2}"/>
+      <geometry>
+        <mesh filename="package://my_robot_description/meshes/collision/wheel.stl" scale="5 5 5"/>
+      </geometry>
+    </collision>
+    <inertial>
+      <mass value="0.25"/>
+      <inertia ixx="0.01" ixy="0.0" ixz="0.0" iyy="0.01" iyz="0.0" izz="0.01"/>
+      <origin xyz="0 0 0"/>
+    </inertial>
+  </link>
+  <joint name="right_rear_wheel_joint" type="continuous">
+    <parent link="base_link"/>
+    <child link="right_rear_wheel"/>
+    <origin xyz="-${0.28-wheel_radius+0.05} -${wheel_separation/2-0.05} -0.1" rpy="0 0 0"/>
+    <axis xyz="0 1 0"/>
+    <dynamics friction="0.0" damping="0.0"/>
   </joint>
   <link name="front_camera">
