Commit message: fix model and rviz

File: src/my_robot_description/models/my_mobile/model.urdf (robot description, URDF)
Before this commit: robot my_mobile, 6 links, 5 joints
Joints:
- joint front_camera_joint: origin xyz=0.3 0 0.25 rpy=0 -${pi/4+0.17453/2} 0 -> xyz=0.3 0 0.25 rpy=0 -0 0
- joint left_rear_wheel_joint: origin xyz=-${0.28-wheel_radius+0.05} ${wheel_separation/2-0.05} -0.1 rpy=0 0 0 -> xyz=-${0.28-wheel_radius+0.05} ${wheel_separation/2-0.05} -0 rpy=0 0 0
- joint left_wheel_joint: origin xyz=${0.28-wheel_radius} ${wheel_separation/2-0.05} 0.3 rpy=0 0 0 -> xyz=${0.28-wheel_radius} ${wheel_separation/2-0.05} 0 rpy=0 0 0
- joint right_rear_wheel_joint: origin xyz=-${0.28-wheel_radius+0.05} -${wheel_separation/2-0.05} -0.1 rpy=0 0 0 -> xyz=-${0.28-wheel_radius+0.05} -${wheel_separation/2-0.05} -0 rpy=0 0 0
- joint right_wheel_joint: origin xyz=${0.28-wheel_radius} -${wheel_separation/2-0.05} 0.3 rpy=0 0 0 -> xyz=${0.28-wheel_radius} -${wheel_separation/2-0.05} 0 rpy=0 0 0

File: src/my_robot_description/urdf/robot_core.xacro (robot description, xacro)
@@ -21,13 +21,13 @@
   <link name="base_link">
     <visual>
-      <origin xyz="0 0 0" rpy="0 -0.0 0"/>
+      <origin xyz="0 0 0" rpy="0 -0  0"/>
       <geometry>
-        <mesh filename="package://my_robot_description/models/my_mobile/meshes/visual/sejongDel_body_origin45.dae" scale="0.00075 0.0005 0.00075"/>
+        <mesh filename="package://my_robot_description/models/my_mobile/meshes/visual/sejongDel_body.dae" scale="0.00075 0.0005 0.00075"/>
       </geometry>
     </visual>
     <collision>
-      <origin xyz="0 0 0" rpy="0 -0.0 0"/>
+      <origin xyz="0 0 0" rpy="0 -0  0"/>
       <geometry>
-        <mesh filename="package://my_robot_description/models/my_mobile/meshes/collision/sejongDel_body_origin45.stl" scale="0.00075 0.0005 0.00075"/>
+        <mesh filename="package://my_robot_description/models/my_mobile/meshes/collision/sejongDel_body.stl" scale="0.00075 0.0005 0.00075"/>
       </geometry>
     </collision>
@@ -60,5 +60,5 @@
     <parent link="base_link"/>
     <child link="left_wheel"/>
-    <origin xyz="${0.28-wheel_radius} ${wheel_separation/2-0.05} 0.3" rpy="0 0 0"/>
+    <origin xyz="${0.28-wheel_radius} ${wheel_separation/2-0.05} 0" rpy="0 0 0"/>
     <axis xyz="0 1 0"/>
   </joint>
@@ -85,5 +85,5 @@
     <parent link="base_link"/>
     <child link="right_wheel"/>
-    <origin xyz="${0.28-wheel_radius} -${wheel_separation/2-0.05} 0.3" rpy="0 0 0"/>
+    <origin xyz="${0.28-wheel_radius} -${wheel_separation/2-0.05} 0" rpy="0 0 0"/>
     <axis xyz="0 1 0"/>
   </joint>
@@ -110,5 +110,5 @@
     <parent link="base_link"/>
     <child link="left_rear_wheel"/>
-    <origin xyz="-${0.28-wheel_radius+0.05} ${wheel_separation/2-0.05} -0.1" rpy="0 0 0"/>
+    <origin xyz="-${0.28-wheel_radius+0.05} ${wheel_separation/2-0.05} -0" rpy="0 0 0"/>
     <axis xyz="0 1 0"/>
     <dynamics friction="0.0" damping="0.0"/>
@@ -136,5 +136,5 @@
     <parent link="base_link"/>
     <child link="right_rear_wheel"/>
-    <origin xyz="-${0.28-wheel_radius+0.05} -${wheel_separation/2-0.05} -0.1" rpy="0 0 0"/>
+    <origin xyz="-${0.28-wheel_radius+0.05} -${wheel_separation/2-0.05} -0" rpy="0 0 0"/>
     <axis xyz="0 1 0"/>
     <dynamics friction="0.0" damping="0.0"/>
@@ -162,5 +162,5 @@
     <parent link="base_link"/>
     <child link="front_camera"/>
-    <origin xyz="0.3 0 0.25" rpy="0 -${pi/4+0.17453/2} 0"/>
+    <origin xyz="0.4 0 0.0" rpy="0 -0 0"/>
   </joint>
   <gazebo reference="front_camera">

Commit message: edit matlab code

File: src/my_robot_description/models/my_mobile/model.urdf (robot description, URDF)
Before this commit: robot my_mobile, 6 links, 5 joints
Joints:
- joint front_camera_joint: origin xyz=0.3 0 0.25 rpy=0 -0 0 -> xyz=0.3 0 -0.05 rpy=0 -0 0

File: src/my_robot_description/urdf/robot_core.xacro (robot description, xacro)
@@ -162,5 +162,5 @@
     <parent link="base_link"/>
     <child link="front_camera"/>
-    <origin xyz="0.4 0 0.0" rpy="0 -0 0"/>
+    <origin xyz="0.3 0 -0.05" rpy="0 -0 0"/>
   </joint>
   <gazebo reference="front_camera">

Commit message: final commit

File: src/my_robot_description/models/my_mobile/model.urdf (robot description, URDF)
Before this commit: robot my_mobile, 6 links, 5 joints
Links:
- added link right_logo, mass 0.001; collision mesh filename=package://my_robot_description/models/my_mobile/meshes/coll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 scale=0.001 0.001 0.001; visual mesh filename=package://my_robot_description/models/my_mobile/meshes/visu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 scale=0.001 0.001 0.001
- added link right_logo_bg, mass 0.001; collision mesh filename=package://my_robot_description/models/my_mobile/meshes/coll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 scale=0.001 0.001 0.001; visual mesh filename=package://my_robot_description/models/my_mobile/meshes/visu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 scale=0.001 0.001 0.001
Joints:
- added joint right_logo_bg_joint: type fixed, parent base_link, child right_logo_bg, origin xyz=0 0 1.0 rpy=0 0 0
- added joint right_logo_joint: type fixed, parent right_logo_bg, child right_logo, origin xyz=0 0 0 rpy=0 0 0

File: src/my_robot_description/urdf/robot_core.xacro (robot description, xacro)
@@ -16,4 +16,5 @@
   </plugin>
 </gazebo>
+  <xacro:property name="pi" value="3.14159265359"/>
   <xacro:property name="wheel_separation" value="0.6"/>
   <xacro:property name="wheel_radius" value="0.1"/>
@@ -38,4 +39,100 @@
     </inertial>
   </link>
+  <link name="right_logo_bg">
+    <visual>
+      <origin xyz="0 0 0" rpy="0 0 0"/>
+      <geometry>
+        <mesh filename="package://my_robot_description/models/my_mobile/meshes/visual/sejongMark_background.dae" scale="0.00075 0.00075 0.00075"/>
+      </geometry>
+    </visual>
+    <collision>
+      <origin xyz="0 0 0" rpy="0 0 0"/>
+      <geometry>
+        <mesh filename="package://my_robot_description/models/my_mobile/meshes/collision/sejongMark_background.stl" scale="0.00075 0.00075 0.00075"/>
+      </geometry>
+    </collision>
+    <inertial>
+      <mass value="0.001"/>
+      <inertia ixx="0.01" ixy="0.0" ixz="0.0" iyy="0.01" iyz="0.0" izz="0.01"/>
+      <origin xyz="0 0 0"/>
+    </inertial>
+  </link>
+  <joint name="right_logo_bg_joint" type="fixed">
+    <parent link="base_link"/>
+    <child link="right_logo_bg"/>
+    <origin xyz="-0.475 0.525 -0.05" rpy="0 0 0"/>
+  </joint>
+  <link name="right_logo">
+    <visual>
+      <origin xyz="0 0 0" rpy="0 0 0"/>
+      <geometry>
+        <mesh filename="package://my_robot_description/models/my_mobile/meshes/visual/sejongMark.dae" scale="0.00075 0.00075 0.00075"/>
+      </geometry>
+    </visual>
+    <collision>
+      <origin xyz="0 0 0" rpy="0 0 0"/>
+      <geometry>
+        <mesh filename="package://my_robot_description/models/my_mobile/meshes/collision/sejongMark.stl" scale="0.00075 0.00075 0.00075"/>
+      </geometry>
+    </collision>
+    <inertial>
+      <mass value="0.001"/>
+      <inertia ixx="0.01" ixy="0.0" ixz="0.0" iyy="0.01" iyz="0.0" izz="0.01"/>
+      <origin xyz="0 0 0"/>
+    </inertial>
+  </link>
+  <joint name="right_logo_joint" type="fixed">
+    <parent link="right_logo_bg"/>
+    <child link="right_logo"/>
+    <origin xyz="0 0.0005 0" rpy="0 0 0"/>
+  </joint>
+  <link name="left_logo_bg">
+    <visual>
+      <origin xyz="0 0 0" rpy="0 0 0"/>
+      <geometry>
+        <mesh filename="package://my_robot_description/models/my_mobile/meshes/visual/sejongMark_background.dae" scale="0.00075 0.00075 0.00075"/>
+      </geometry>
+    </visual>
+    <collision>
+      <origin xyz="0 0 0" rpy="0 0 0"/>
+      <geometry>
+        <mesh filename="package://my_robot_description/models/my_mobile/meshes/collision/sejongMark_background.stl" scale="0.00075 0.00075 0.00075"/>
+      </geometry>
+    </collision>
+    <inertial>
+      <mass value="0.001"/>
+      <inertia ixx="0.01" ixy="0.0" ixz="0.0" iyy="0.01" iyz="0.0" izz="0.01"/>
+      <origin xyz="0 0 0"/>
+    </inertial>
+  </link>
+  <joint name="left_logo_bg_joint" type="fixed">
+    <parent link="base_link"/>
+    <child link="left_logo_bg"/>
+    <origin xyz="0.475 -0.525 -0.05" rpy="0 0 ${pi}"/>
+  </joint>
+  <link name="left_logo">
+    <visual>
+      <origin xyz="0 0 0" rpy="0 0 0"/>
+      <geometry>
+        <mesh filename="package://my_robot_description/models/my_mobile/meshes/visual/sejongMark.dae" scale="0.00075 0.00075 0.00075"/>
+      </geometry>
+    </visual>
+    <collision>
+      <origin xyz="0 0 0" rpy="0 0 0"/>
+      <geometry>
+        <mesh filename="package://my_robot_description/models/my_mobile/meshes/collision/sejongMark.stl" scale="0.00075 0.00075 0.00075"/>
+      </geometry>
+    </collision>
+    <inertial>
+      <mass value="0.001"/>
+      <inertia ixx="0.01" ixy="0.0" ixz="0.0" iyy="0.01" iyz="0.0" izz="0.01"/>
+      <origin xyz="0 0 0"/>
+    </inertial>
+  </link>
+  <joint name="left_logo_joint" type="fixed">
+    <parent link="left_logo_bg"/>
+    <child link="left_logo"/>
+    <origin xyz="0 0.0005 0" rpy="0 0 0"/>
+  </joint>
   <link name="left_wheel">
     <visual>
